File: GD5434.kicad_pcb (KiCad board)
At the start: 4 copper layers, 157.5 x 88.2 mm, 132 parts, among them J0 Bus_ISA_16bit, J1 DB15_Female_HighDensity_Mount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, J2 Feature connector, U1 CL-GD5434-ISA, U10 7438, U11 93CxxA, U12 NUP4202, U13 NUP4202, U2 IS41C16257, U3 IS41C16257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

Commit message: Add files via upload
fixed 74LS245 connections
Parts:
- removed G*** (x2): LOGO, owl:owl-20mm
- added REF**: owl-20mm-mask-base, owl:owl-20mm-mask-base, B.Cu at (94.6, 48.5)
- added REF**: owl-20mm-mask, owl:owl-20mm-mask, B.Cu at (94.7, 48.5)
- added REF**: owl-20mm-mask-base, owl:owl-20mm-mask-base, F.Cu at (215.0, 36.5)
- added REF**: owl-20mm-mask, owl:owl-20mm-mask, F.Cu at (215.0, 36.5)
- U12, U13: value NUP4202 -> TPD4E1U06DBVR; footprint Package_TO_SOT_SMD:SOT-363_SC-70-6 -> Package_TO_SOT_SMD:SOT-23-6_Handsoldering
- moved JP1 15.2 mm to (190.6, 99.5)
- moved C67 14.5 mm to (206.3, 95.5), turned to 270 degrees
- moved C66 14.3 mm to (206.1, 88.0), turned to 90 degrees
- moved R23 2.03 mm to (167.9, 84.9)
- moved C25 1.92 mm to (167.9, 86.9)
- moved U12 1.72 mm to (212.6, 60.8)
- moved U6 1.33 mm to (200.3, 98.2), turned to 0 degrees
- moved U7 0.96 mm to (198.4, 84.4), turned to 270 degrees
- moved U13 0.86 mm to (212.6, 69.0)
- moved C10 0.80 mm to (201.6, 57.2)
- moved C11 0.80 mm to (201.6, 61.1)
- moved C13 0.80 mm to (205.4, 57.2)
- moved C14 0.80 mm to (205.4, 61.1)
- moved C15 0.80 mm to (205.4, 65.1)
- moved C16 0.80 mm to (208.4, 56.2)
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Connections:
- U12 pad 1: Net-(C16-Pad1) -> (no net)
- U12 pad 3: (no net) -> Net-(C18-Pad1)
- U12 pad 4: Net-(C18-Pad1) -> Net-(C17-Pad1)
- U12 pad 5: VCC -> (no net)
- U12 pad 6: Net-(C17-Pad1) -> Net-(C16-Pad1)
- U13 pad 5: VCC -> (no net)
- U6 pad 1: /RESET_DRV -> GND
- U6 pad 2: Net-(R23-Pad2) -> (no net)
- U6 pad 5: GND -> /RESET_DRV
- U6 pad 6: (no net) -> Net-(R23-Pad2)
- U7 pad 2: /SD7 -> /SD0
- U7 pad 3: /SD6 -> /SD1
- U7 pad 4: /SD5 -> /SD2
- U7 pad 5: /SD4 -> /SD3
- U7 pad 6: /SD3 -> /SD4
- U7 pad 7: /SD2 -> /SD5
- U7 pad 8: /SD1 -> /SD6
- U7 pad 9: /SD0 -> /SD7
Routing:
- net BLUE: track 62.8 -> 37.7 mm
- net /IRQ: track 59.1 -> 43.2 mm
- net GND: track 236.8 -> 249.1 mm, vias 257 -> 258
- net Net-(U7-Pad18): track 10.6 -> 18.4 mm
- net /RESET_DRV: track 12.0 -> 19.3 mm
- net Net-(U7-Pad13): track 9.44 -> 16.6 mm
- net Net-(U7-Pad17): track 7.47 -> 14.6 mm
- net Net-(J0-Pad4): track 12.7 -> 19.6 mm
- net Net-(U7-Pad14): track 6.11 -> 13.0 mm
- net /EROM: track 50.3 -> 57.1 mm
- net /SD0: track 82.2 -> 88.8 mm
- net Net-(U7-Pad15): track 10.4 -> 16.5 mm
- net Net-(U7-Pad16): track 10.7 -> 16.5 mm
- net /SD6: track 69.9 -> 75.6 mm
- net /SD3: track 74.9 -> 80.0 mm
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Other:
- net class data added: clearance 0.15, trace_width 0.1524, via_dia 0.6, via_drill 0.3
- board text added: "JLCJLCJLCJLC"
- board text added: "JP1 - IRQ2/9 enable JP2 - Zero WS JP3 - ROM section select JP4 & R5 - 64K ROM"
- board text added: "Pine"
- board text removed: "JP1 - IRQ2/9 enable JP2 - Zero WS JP3 - ROM section select JP4 & R8 - 64K ROM"

Commit message: Add files via upload
Few updates + BOM
Parts:
- added NT1: Net-Tie_2, NetTie:NetTie-2_SMD_Pad0.5mm, B.Cu at (165.2, 55.4)
- moved R50 1.09 mm to (137.1, 49.1)
Connections:
- U1 pad 104: (no net) -> Net-(NT1-Pad2)
Routing:
- net /SA2: track 68.7 -> 71.6 mm
- net /SA3: track 64.6 -> 67.4 mm
- net /SA5: track 57.1 -> 59.9 mm
- net Net-(NT1-Pad2): track 0.00 -> 2.66 mm, vias 0 -> 1
- net GND: track 249.1 -> 251.5 mm, vias 258 -> 266
- net /SA4: track 62.0 -> 63.9 mm
- net VCC: track 129.6 -> 128.4 mm
- net /CAS2: track 7.58 -> 6.90 mm
- net Net-(C68-Pad1): track 16.4 -> 17.1 mm, vias 1 -> 2
- net VDD: track 37.0 -> 37.6 mm, vias 15 -> 16
Other:
- rule solder_mask_min_width: 0.0508 -> 0.2
