File: GD5434.sch (KiCad schematic (older format))
At the start: 130 parts, among them J0 Bus_ISA_16bit, J1 DB15_Female_HighDensity_Mount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, J2 Feature connector, U1 CL-GD5434-ISA, U10 7438, U11 93CxxA, U12 NUP4202, U13 NUP4202, U2 IS41C16257, U3 IS41C16257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

Commit message: Add files via upload
fixed 74LS245 connections
Parts:
- U12, U13: value NUP4202 -> TPD4E1U06DBVR; footprint Package_TO_SOT_SMD:SOT-363_SC-70-6 -> Package_TO_SOT_SMD:SOT-23-6_Handsoldering
Connections:
- net GND: now also U6.1; no longer U6.5
- net RESET_DRV: now also U6.5; no longer U6.1
- net SD0: now also U7.2 (A0); no longer U7.9 (A7)
- net SD1: now also U7.3 (A1); no longer U7.8 (A6)
- net SD2: now also U7.4 (A2); no longer U7.7 (A5)
- net SD3: now also U7.5 (A3); no longer U7.6 (A4)
- net SD4: now also U7.6 (A4); no longer U7.5 (A3)
- net SD5: now also U7.7 (A5); no longer U7.4 (A2)
- net SD6: now also U7.8 (A6); no longer U7.3 (A1)
- net SD7: now also U7.9 (A7); no longer U7.2 (A0)
- net VCC: no longer U12.5, U13.5
- net at C16.1, J1.1, L4.2: now also U12.6; no longer U12.1
- net at C17.1, J1.2, L5.2: now also U12.4; no longer U12.6
- net at C18.1, J1.3, L6.2: now also U12.3; no longer U12.4
- net at U6.2: no longer R23.2
- net at U6.6: now also R23.2
- no-connect marks 54 -> 56
Other:
- moved on the sheet: C1, C10, C11, C12, C13, C14, C15, C16, C17, C18, C2, C20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

Commit message: Add files via upload
Few updates + BOM
Parts:
- added NT1: Net-Tie_2, NetTie:NetTie-2_SMD_Pad0.5mm, symbol Device:Net-Tie_2
Connections:
- net GND: now also U1.208 (VSS13), NT1.1; no longer U1.104 (VSS6)
- new net: NT1.2, U1.104 (VSS6)
Changed lines of the file:
@@
 	10100 11550 10100 11650
 Connection ~ 10100 11650
-Wire Wire Line
-	10150 11450 10100 11450
-Wire Wire Line
-	10100 11450 10100 11550
 Connection ~ 10100 11550
 Wire Wire Line
 	10150 11350 10100 11350
 Wire Wire Line
-	10100 11350 10100 11450
-Connection ~ 10100 11450
-Wire Wire Line
 	10150 11250 10100 11250
 Wire Wire Line
@@
 	11800 7000 11850 7000
 NoConn ~ 7050 12500
-$Comp
-L gd5434:CL-GD5434-ISA U1
-U 1 1 5E737213
-P 14650 11550
-F 0 "U1" H 18000 10850 50  0000 L CNN
-F 1 "CL-GD5434-ISA" H 17750 10700 50  0000 L CNN
-F 2 "Package_QFP:PQFP-208_28x28mm_P0.5mm" H 14700 11450 50  0001 C CNN
-F 3 "" H 14650 11550 50  0001 C CNN
-	1    14650 11550
-	1    0    0    -1
-$EndComp
 NoConn ~ 17700 9650
 $Comp
@@
 Wire Wire Line
 	26200 8950 26200 10250
+Connection ~ 26200 10250
+Wire Wire Line
+	26200 10250 26300 10250
+Wire Wire Line
+	10100 12050 10100 12150
+Wire Wire Line
+	10100 12150 10150 12150
+Connection ~ 10100 12050
+$Comp
+L Device:Net-Tie_2 NT1
+U 1 1 5F3D9040
+P 9700 11450
+F 0 "NT1" H 9700 11631 50  0000 C CNN
+F 1 "Net-Tie_2" H 9700 11540 50  0000 C CNN
+F 2 "NetTie:NetTie-2_SMD_Pad0.5mm" H 9700 11450 50  0001 C CNN
+F 3 "~" H 9700 11450 50  0001 C CNN
+	1    9700 11450
+	1    0    0    -1
+$EndComp
+Wire Wire Line
+	10100 11350 10100 11550
+Wire Wire Line
+	10150 11450 9800 11450
+Wire Wire Line
+	9600 11450 9300 11450
+Wire Wire Line
+	9300 11450 9300 10600
+$Comp
+L gd5434:CL-GD5434-ISA U1
+U 1 1 5E737213
+P 14650 11550
+F 0 "U1" H 18000 10850 50  0000 L CNN
+F 1 "CL-GD5434-ISA" H 17750 10700 50  0000 L CNN
+F 2 "Package_QFP:PQFP-208_28x28mm_P0.5mm" H 14700 11450 50  0001 C CNN
+F 3 "" H 14650 11550 50  0001 C CNN
+	1    14650 11550
+	1    0    0    -1
+$EndComp
 Wire Bus Line
 	11200 13800 11200 14900
@@
 Wire Bus Line
 	10400 9350 19100 9350
-Connection ~ 26200 10250
-Wire Wire Line
-	26200 10250 26300 10250
 $EndSCHEMATC
